Commit message: feat: add multi-object visual grasp selection

File: packages/panda_moveit_config/config/panda.ros2_control.xacro (robot description, xacro)
@@ -45,5 +45,5 @@
   <xacro:macro
     name="panda_gz_ros2_control"
-    params="initial_positions_file controllers_file assisted_grasp">
+    params="initial_positions_file controllers_file assisted_grasp workpiece_count">
     <xacro:property
       name="initial_positions"
@@ -118,4 +118,5 @@
          Gazebo Sim and never gazebo_ros2_control / Gazebo Classic. -->
     <xacro:if value="${assisted_grasp}">
+      <xacro:macro name="detachable_workpiece" params="suffix child_model child_link">
       <gazebo>
         <plugin
@@ -123,11 +124,17 @@
           name="ignition::gazebo::systems::DetachableJoint">
           <parent_link>panda_hand</parent_link>
-          <child_model>cube</child_model>
-          <child_link>cube_link</child_link>
-          <detach_topic>/panda/detachable_joint/detach</detach_topic>
-          <attach_topic>/panda/detachable_joint/attach</attach_topic>
-          <output_topic>/panda/detachable_joint/state</output_topic>
+          <child_model>${child_model}</child_model>
+          <child_link>${child_link}</child_link>
+          <detach_topic>/panda/detachable_joint${suffix}/detach</detach_topic>
+          <attach_topic>/panda/detachable_joint${suffix}/attach</attach_topic>
+          <output_topic>/panda/detachable_joint${suffix}/state</output_topic>
         </plugin>
       </gazebo>
+      </xacro:macro>
+      <xacro:detachable_workpiece suffix="" child_model="cube" child_link="cube_link" />
+      <xacro:if value="${int(workpiece_count) == 3}">
+        <xacro:detachable_workpiece suffix="_1" child_model="cube_1" child_link="cube_1_link" />
+        <xacro:detachable_workpiece suffix="_2" child_model="cube_2" child_link="cube_2_link" />
+      </xacro:if>
     </xacro:if>
     <gazebo reference="panda_leftfinger"><mu1>1.2</mu1><mu2>1.2</mu2></gazebo>

File: packages/panda_moveit_config/config/panda.urdf.xacro (robot description, xacro)
@@ -7,4 +7,5 @@
   <xacro:arg name="controllers_file" default="" />
   <xacro:arg name="assisted_grasp" default="true" />
+  <xacro:arg name="workpiece_count" default="1" />
   <!-- This is the only Panda robot_description entry point for mock and Gazebo. -->
   <xacro:include filename="panda_description.urdf.xacro" />
@@ -54,5 +55,6 @@
       initial_positions_file="$(arg initial_positions_file)"
       controllers_file="$(arg controllers_file)"
-      assisted_grasp="$(arg assisted_grasp)" />
+      assisted_grasp="$(arg assisted_grasp)"
+      workpiece_count="$(arg workpiece_count)" />
   </xacro:if>
 </robot>
